File: board/wifilamp2a.brd (EAGLE design)
At the start: 25.4 x 39.4 mm, 6 parts

Commit message: [board] Update board to rev 2.1
Parts:
- added JP1: (no value), SparkFun-Jumpers:SMT-JUMPER_3_1-NC_TRACE_NO-SILK
Connections:
- new net N$1: JP1.1, U$1.D1
- new net N$3: JP1.2, LED.2
- net N$2: now also JP1.3, U$1.D4; no longer LED.2, U$1.D1
Routing:
- net N$3: track 0.00 -> 28.5 mm
- net N$2: track 31.7 -> 5.23 mm
- net N$1: track 0.00 -> 5.23 mm
- net GND: track 65.6 -> 66.6 mm
Other:
- board text added: "v2.1"
